File: sch/main-uno.kicad_sch (KiCad schematic)
At the start: 2 parts, among them J1 Analog, J2 Digital

Commit message: tmp
Connections:
- net *D10/SS renamed RELAY_HIGH_POERT
- net *D5 renamed SWITCH_4 -> SWITCH_LOW_POWER_PERMAMENT_ON
- net *D6 renamed SWITCH_3 -> SWITCH_HIGH_POWER_PERMAMENT_ON
- net *D9 renamed RELAY_RADIO
- net A7 renamed BATTERY_VOLTAGE
- net BATTERY_CHARGING renamed RELAY_CHARGING
- net D7 renamed SWITCH_2 -> SWITCH_RADIO_PERMAMENT_ON
- net D8 renamed SWITCH_1 -> SWITCH_RADIO_AUTO_START
- net SUPPLY_RADIO renamed RELAY_LOW_POWER
Changed lines of the file:
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@@
 (kicad_sch
-	(version 20231120)
+	(version 20250114)
 	(generator "eeschema")
-	(generator_version "8.0")
+	(generator_version "9.0")
 	(paper "A4")
 	(title_block
@@
 	(wire
 		(pts
-			(xy 149.86 50.8) (xy 165.1 50.8)
-		)
-		(stroke
-			(width 0)
-			(type solid)
-		)
-	)
-	(wire
-		(pts
-			(xy 149.86 55.88) (xy 165.1 55.88)
-		)
-		(stroke
-			(width 0)
-			(type solid)
-		)
-	)
-	(wire
-		(pts
-			(xy 149.86 58.42) (xy 165.1 58.42)
+			(xy 149.86 50.8) (xy 168.91 50.8)
+		)
+		(stroke
+			(width 0)
+			(type solid)
+		)
+	)
+	(wire
+		(pts
+			(xy 149.86 55.88) (xy 168.91 55.88)
+		)
+		(stroke
+			(width 0)
+			(type solid)
+		)
+	)
+	(wire
+		(pts
+			(xy 149.86 58.42) (xy 168.91 58.42)
 		)
 		(stroke
@@
 	(wire
 		(pts
-			(xy 149.86 63.5) (xy 165.1 63.5)
+			(xy 149.86 63.5) (xy 168.91 63.5)
 		)
 		(stroke
@@
 	(wire
 		(pts
-			(xy 149.86 60.96) (xy 165.1 60.96)
+			(xy 149.86 60.96) (xy 168.91 60.96)
 		)
 		(stroke
@@
 	(wire
 		(pts
-			(xy 111.76 71.12) (xy 129.54 71.12)
+			(xy 109.22 71.12) (xy 129.54 71.12)
 		)
 		(stroke
@@
 	(wire
 		(pts
-			(xy 149.86 53.34) (xy 165.1 53.34)
+			(xy 149.86 53.34) (xy 168.91 53.34)
 		)
 		(stroke
@@
 	(wire
 		(pts
-			(xy 110.49 68.58) (xy 129.54 68.58)
+			(xy 109.22 68.58) (xy 129.54 68.58)
 		)
 		(stroke
@@
 	(label "D4"
 		(at 165.1 66.04 180)
-		(fields_autoplaced yes)
 		(effects
 			(font
@@
 	(label "*D5"
 		(at 165.1 63.5 180)
-		(fields_autoplaced yes)
 		(effects
 			(font
@@
 	(label "A2"
 		(at 111.76 58.42 0)
-		(fields_autoplaced yes)
 		(effects
 			(font
@@
 	(label "D7"
 		(at 165.1 58.42 180)
-		(fields_autoplaced yes)
 		(effects
 			(font
@@
 	(label "D13{slash}SCK"
 		(at 111.76 45.72 0)
-		(fields_autoplaced yes)
 		(effects
 			(font
@@
 	(label "A7"
 		(at 111.76 71.12 0)
-		(fields_autoplaced yes)
 		(effects
 			(font
@@
 	(label "*D6"
 		(at 165.1 60.96 180)
-		(fields_autoplaced yes)
 		(effects
 			(font
@@
 	(label "*D11{slash}MOSI"
 		(at 165.1 48.26 180)
-		(fields_autoplaced yes)
 		(effects
 			(font
@@
 	(label "A1"
 		(at 111.76 55.88 0)
-		(fields_autoplaced yes)
 		(effects
 			(font
@@
 	(label "A4{slash}SDA"
 		(at 111.76 63.5 0)
-		(fields_autoplaced yes)
 		(effects
 			(font
@@
 	(label "A5{slash}SCL"
 		(at 111.76 66.04 0)
-		(fields_autoplaced yes)
 		(effects
 			(font
@@
 	(label "A3"
 		(at 111.76 60.96 0)
-		(fields_autoplaced yes)
 		(effects
 			(font
@@
 	(label "~{RESET}"
 		(at 165.1 76.2 180)
-		(fields_autoplaced yes)
 		(effects
 			(font
@@
 	(label "~{RESET}"
 		(at 111.76 76.2 0)
-		(fields_autoplaced yes)
 		(effects
 			(font
@@
 	(label "A6"
 		(at 111.76 68.58 0)
-		(fields_autoplaced yes)
 		(effects
 			(font
@@
 	(label "A0"
 		(at 111.76 53.34 0)
-		(fields_autoplaced yes)
 		(effects
 			(font
@@
 	(label "*D9"
 		(at 165.1 53.34 180)
-		(fields_autoplaced yes)
 		(effects
 			(font
@@
 	(label "*D3"
 		(at 165.1 68.58 180)
-		(fields_autoplaced yes)
 		(effects
 			(font
@@
 	(label "D2"
 		(at 165.1 71.12 180)
-		(fields_autoplaced yes)
 		(effects
 			(font
@@
 	(label "D8"
 		(at 165.1 55.88 180)
-		(fields_autoplaced yes)
 		(effects
 			(font
@@
 	(label "D1{slash}TX"
 		(at 165.1 81.28 180)
-		(fields_autoplaced yes)
 		(effects
 			(font
@@
 	(label "D0{slash}RX"
 		(at 165.1 78.74 180)
-		(fields_autoplaced yes)
 		(effects
 			(font
@@
 	(label "AREF"
 		(at 111.76 50.8 0)
-		(fields_autoplaced yes)
 		(effects
 			(font
@@
 	(label "*D10{slash}SS"
 		(at 165.1 50.8 180)
-		(fields_autoplaced yes)
 		(effects
 			(font
@@
 	(label "D12{slash}MISO"
 		(at 165.1 45.72 180)
+		(effects
+			(font
+				(size 1.27 1.27)
+			)
+			(justify right bottom)
+		)
+	)
+	(global_label "BATTERY_VOLTAGE"
+		(shape input)
+		(at 109.22 71.12 180)
 		(fields_autoplaced yes)
 		(effects
@@
 				(size 1.27 1.27)
 			)
-			(justify right bottom)
-		)
-	)
-	(global_label "BATTERY_CHARGING"
+			(justify right)
+		)
+		(property "Intersheetrefs" "${INTERSHEET_REFS}"
+			(at 90.7535 71.12 0)
+			(effects
+				(font
+					(size 1.27 1.27)
+				)
+				(justify right)
+				(hide yes)
+			)
+		)
+	)
+	(global_label "RELAY_CHARGING"
 		(shape input)
 		(at 168.91 45.72 0)
@@
 		)
 		(property "Intersheetrefs" "${INTERSHEET_REFS}"
-			(at 188.8568 45.72 0)
+			(at 186.4149 45.72 0)
+			(effects
+				(font
+					(size 1.27 1.27)
+				)
+				(justify left)
+				(hide yes)
+			)
+		)
+	)
+	(global_label "RELAY_HIGH_POERT"
+		(shape input)
+		(at 168.91 50.8 0)
+		(fields_autoplaced yes)
+		(effects
+			(font
+				(size 1.27 1.27)
+			)
+			(justify left)
+		)
+		(property "Intersheetrefs" "${INTERSHEET_REFS}"
+			(at 188.2711 50.8 0)
+			(effects
+				(font
+					(size 1.27 1.27)
+				)
+				(justify left)
+				(hide yes)
+			)
+		)
+	)
+	(global_label "SWITCH_2 -> SWITCH_RADIO_PERMAMENT_ON"
+		(shape input)
+		(at 168.91 58.42 0)
+		(fields_autoplaced yes)
+		(effects
+			(font
+				(size 1.27 1.27)
+			)
+			(justify left)
+		)
+		(property "Intersheetrefs" "${INTERSHEET_REFS}"
+			(at 209.9297 58.42 0)
 			(effects
 				(font
@@
 	(global_label "CAR_VOLTAGE"
 		(shape input)
-		(at 110.49 68.58 180)
+		(at 109.22 68.58 180)
 		(fields_autoplaced yes)
 		(effects
@@
 		)
 		(property "Intersheetrefs" "${INTERSHEET_REFS}"
-			(at 95.8388 68.58 0)
+			(at 94.5688 68.58 0)
 			(effects
 				(font
@@
 		)
 	)
-	(global_label "SUPPLY_RADIO"
+	(global_label "RELAY_LOW_POWER"
 		(shape input)
 		(at 168.91 48.26 0)
@@
 		)
 		(property "Intersheetrefs" "${INTERSHEET_REFS}"
-			(at 184.2275 48.26 0)
+			(at 188.6843 48.26 0)
+			(effects
+				(font
+					(size 1.27 1.27)
+				)
+				(justify left)
+				(hide yes)
+			)
+		)
+	)
+	(global_label "SWITCH_1 -> SWITCH_RADIO_AUTO_START"
+		(shape input)
+		(at 168.91 55.88 0)
+		(fields_autoplaced yes)
+		(effects
+			(font
+				(size 1.27 1.27)
+			)
+			(justify left)
+		)
+		(property "Intersheetrefs" "${INTERSHEET_REFS}"
+			(at 206.3849 55.88 0)
+			(effects
+				(font
+					(size 1.27 1.27)
+				)
+				(justify left)
+				(hide yes)
+			)
+		)
+	)
+	(global_label "SWITCH_4 -> SWITCH_LOW_POWER_PERMAMENT_ON"
+		(shape input)
+		(at 168.91 63.5 0)
+		(fields_autoplaced yes)
+		(effects
+			(font
+				(size 1.27 1.27)
+			)
+			(justify left)
+		)
+		(property "Intersheetrefs" "${INTERSHEET_REFS}"
+			(at 215.4548 63.5 0)
+			(effects
+				(font
+					(size 1.27 1.27)
+				)
+				(justify left)
+				(hide yes)
+			)
+		)
+	)
+	(global_label "RELAY_RADIO"
+		(shape input)
+		(at 168.91 53.34 0)
+		(fields_autoplaced yes)
+		(effects
+			(font
+				(size 1.27 1.27)
+			)
+			(justify left)
+		)
+		(property "Intersheetrefs" "${INTERSHEET_REFS}"
+			(at 183.1592 53.34 0)
+			(effects
+				(font
+					(size 1.27 1.27)
+				)
+				(justify left)
+				(hide yes)
+			)
+		)
+	)
+	(global_label "SWITCH_3 -> SWITCH_HIGH_POWER_PERMAMENT_ON"
+		(shape input)
+		(at 168.91 60.96 0)
+		(fields_autoplaced yes)
+		(effects
+			(font
+				(size 1.27 1.27)
+			)
+			(justify left)
+		)
+		(property "Intersheetrefs" "${INTERSHEET_REFS}"
+			(at 215.6967 60.96 0)
 			(effects
 				(font
@@
 		)
 	)
+	(embedded_fonts no)
 )
